File: PCB/Penguin_Paddle/Penguin_Paddle.kicad_pcb (KiCad board)
At the start: 2 copper layers, 64.2 x 68.9 mm, 17 parts, among them J1 Conn_01x01_Socket, J2 AudioPlug3, J3 Conn_01x01_Socket, Q1 NPN, SW1 SW_SPST, SW2 SW_SPST, U1 XIAO-ESP32-S3-DIP

Commit message: Cleaned folders (frogot to commit this a few days ago)
Parts:
- added ?: , , B.Cu at (177.2, 124.2)
- added REF**: TestPoint_THTPad_1.0x1.0mm_Drill0.5mm, TestPoint:TestPoint_THTPad_1.0x1.0mm_Drill0.5mm, F.Cu at (175.9, 105.0)
- added REF**: TestPoint_THTPad_1.0x1.0mm_Drill0.5mm, TestPoint:TestPoint_THTPad_1.0x1.0mm_Drill0.5mm, B.Cu at (178.4, 105.1)
- added TP2: TestPoint, Custom:Copper Pad, F.Cu at (182.7, 103.7)
- added mouse-bite-1mm-3mm: VAL**, PCB:mouse-bite-1mm-3mm, F.Cu at (191.6, 118.1)
Other:
- board size 64.2 x 68.9 mm -> 93.2 x 68.9 mm
