File: Penguin_Paddle_Files/_autosave-Penguin_Paddle.kicad_pcb (KiCad board)
At the start: 2 copper layers, 64.2 x 68.9 mm, 15 parts, among them J1 Conn_01x01_Socket, J2 AudioPlug3, J3 Conn_01x01_Socket, Q1 NPN, SW1 SW_SPST, SW2 SW_SPST, U1 XIAO-ESP32-S3-DIP

Commit message: Cleaned folders (frogot to commit this a few days ago)
Parts:
- added ?: , , B.Cu at (177.2, 124.2)
- added REF**: MountingHole_2.1mm, MountingHole:MountingHole_2.1mm, F.Cu at (224.5, 142.9)
- added REF**: TestPoint_THTPad_1.0x1.0mm_Drill0.5mm, TestPoint:TestPoint_THTPad_1.0x1.0mm_Drill0.5mm, F.Cu at (175.9, 105.0)
- added REF**: MountingHole_2.1mm, MountingHole:MountingHole_2.1mm, F.Cu at (224.5, 126.3)
- added REF**: TestPoint_THTPad_1.0x1.0mm_Drill0.5mm, TestPoint:TestPoint_THTPad_1.0x1.0mm_Drill0.5mm, B.Cu at (178.4, 105.1)
- added TP2: TestPoint, Custom:Copper Pad, F.Cu at (182.7, 103.7)
- added mouse-bite-1mm-3mm: VAL**, PCB:mouse-bite-1mm-3mm, F.Cu at (191.6, 118.1)
- RV1, RV2: footprint Potentiometer_THT:Potentiometer_Vishay_T73YP_Vertical -> Potentiometer_THT:Potentiometer_TT_P0915N
- moved RV2 6.30 mm to (197.4, 110.0)
- moved SW2 5.06 mm to (212.7, 91.8)
- moved LS1 4.16 mm to (202.2, 90.6)
- moved RV1 4.13 mm to (212.3, 109.9)
- moved SW1 4.06 mm to (212.9, 84.9)
Routing:
- net Net-(U1-GPIO5/D4/I2C_SDA): track 23.2 -> 34.2 mm
- net Net-(U1-GPIO9/D5/I2C_SCL): track 11.1 -> 18.0 mm
- net +3V3: track 78.3 -> 71.6 mm
- net Net-(SW1-B): track 11.0 -> 13.4 mm
- net Net-(JP2-B): track 23.9 -> 22.2 mm
- net Net-(SW2-B): track 14.7 -> 13.4 mm
- net Net-(Q1-B): track 8.16 -> 9.33 mm
- net Net-(U1-GPIO1/D0/A0): track 23.9 -> 24.7 mm
- net Net-(J1-Pin_1): track 25.9 -> 25.3 mm
Other:
- board size 64.2 x 68.9 mm -> 93.2 x 68.9 mm
