File: Penguin_Paddle_Files/Penguin_Paddle.kicad_pcb (KiCad board)
At the start: 2 copper layers, 66.7 x 70.7 mm, 11 parts, among them J2 Audio Plug, Q1 NPN, SW1 SW_SPST, SW2 SW_SPDT, U1 XIAO-ESP32-S3-DIP

Commit message: Cleaned folders (frogot to commit this a few days ago)
Parts:
- added ?: , , B.Cu at (177.2, 124.2)
- added J1: Conn_01x01_Socket, Connector_Wire:SolderWire-0.1sqmm_1x01_D0.4mm_OD1mm, F.Cu at (227.2, 113.5)
- added J3: Conn_01x01_Socket, Connector_Wire:SolderWire-0.1sqmm_1x01_D0.4mm_OD1mm, F.Cu at (221.4, 113.5)
- added JP1: SolderJumper_2_Open, Jumper:SolderJumper-2_P1.3mm_Open_Pad1.0x1.5mm, F.Cu at (221.3, 117.4)
- added JP2: SolderJumper_2_Open, Jumper:SolderJumper-2_P1.3mm_Open_Pad1.0x1.5mm, F.Cu at (227.2, 117.4)
- added REF**: MountingHole_2.1mm, MountingHole:MountingHole_2.1mm, F.Cu at (224.5, 142.9)
- added REF**: TestPoint_THTPad_1.0x1.0mm_Drill0.5mm, TestPoint:TestPoint_THTPad_1.0x1.0mm_Drill0.5mm, F.Cu at (175.9, 105.0)
- added REF**: MountingHole_2.1mm, MountingHole:MountingHole_2.1mm, F.Cu at (224.5, 126.3)
- added REF**: TestPoint_THTPad_1.0x1.0mm_Drill0.5mm, TestPoint:TestPoint_THTPad_1.0x1.0mm_Drill0.5mm, B.Cu at (178.4, 105.1)
- added TP2: TestPoint, Custom:Copper Pad, F.Cu at (182.7, 103.7)
- added mouse-bite-1mm-3mm: VAL**, PCB:mouse-bite-1mm-3mm, F.Cu at (191.6, 118.1)
- J2: value Audio Plug -> AudioPlug3
- LS1: value Piezo Buzzer -> PS1240P02BT
- RV1, RV2: value Potentiometer -> R_Potentiometer; footprint Potentiometer_THT:Potentiometer_Vishay_T73YP_Vertical -> Potentiometer_THT:Potentiometer_TT_P0915N
- SW1: footprint Button_Switch_THT:SW_DIP_SPSTx01_Slide_9.78x4.72mm_W7.62mm_P2.54mm -> Button_Switch_THT:SW_Slide_SPDT_Straight_CK_OS102011MS2Q
- SW2: value SW_SPDT -> SW_SPST
- TP1, TP2: value Copper Pad -> TestPoint
- moved RV2 6.30 mm to (197.4, 110.0)
- moved SW2 5.06 mm to (212.7, 91.8)
- moved LS1 4.16 mm to (202.2, 90.6)
- moved RV1 4.13 mm to (212.3, 109.9)
- moved SW1 3.89 mm to (212.9, 84.9)
- moved TP1 2.01 mm to (251.1, 110.2)
- moved TP2 1.72 mm to (211.5, 110.7)
Connections:
- SW2 pad 1: Net-(SW2-A) -> +3V3
- SW2 pad 2: GND -> Net-(SW2-B)
- SW2 pad 3: +3V3 -> (no net)
- TP1 pad 1: Net-(U1-GPIO8/D9/A9/MISO) -> Net-(JP2-B)
- TP2 pad 1: Net-(U1-GPIO7/D8/A8/SCK) -> Net-(JP1-B)
- U1 pad 10: Net-(U1-GPIO8/D9/A9/MISO) -> Net-(J3-Pin_1)
- U1 pad 4: Net-(SW2-A) -> Net-(SW2-B)
- U1 pad 9: Net-(U1-GPIO7/D8/A8/SCK) -> Net-(J1-Pin_1)
Routing:
- net Net-(U1-GPIO7/D8/A8/SCK): track 66.3 -> 0.00 mm
- net Net-(U1-GPIO8/D9/A9/MISO): track 39.0 -> 0.00 mm
- net Net-(J3-Pin_1): track 0.00 -> 29.5 mm
- net Net-(J1-Pin_1): track 0.00 -> 25.3 mm
- net Net-(JP2-B): track 0.00 -> 22.2 mm
- net Net-(JP1-B): track 0.00 -> 20.8 mm
- net Net-(SW2-A): track 16.7 -> 0.00 mm
- net Net-(SW2-B): track 0.00 -> 13.4 mm
- net Net-(U1-GPIO5/D4/I2C_SDA): track 23.2 -> 34.2 mm
- net Net-(U1-GPIO9/D5/I2C_SCL): track 11.1 -> 18.0 mm
- net Net-(SW1-B): track 7.02 -> 13.4 mm
- net GND: track 86.3 -> 88.4 mm
- net Net-(U1-GPIO1/D0/A0): track 23.3 -> 24.7 mm
- net +3V3: track 72.8 -> 71.6 mm
- net Net-(Q1-B): track 8.16 -> 9.33 mm
Other:
- board size 66.7 x 70.7 mm -> 93.2 x 68.9 mm

Commit message: Finished Code, Switched to Mircopython, updated Gerbers
Parts:
- removed ?: , 
- removed the REF** at (175.9, 105.0)
- removed the REF** at (178.4, 105.1)
- removed the TP2 at (182.7, 103.7)
- removed mouse-bite-1mm-3mm: VAL**, PCB:mouse-bite-1mm-3mm
Other:
- board size 93.2 x 68.9 mm -> 64.2 x 68.9 mm
